File: hw-dartsout.kicad_sch (KiCad schematic)
At the start: 64 parts, among them IC1 FXOS8700CQ, J1 Conn_01x02_Pin, J2 Conn_01x04_Pin, J3 Conn_01x03_Pin, J4 Conn_01x10_Socket, J5 Conn_01x10_Socket, J6 USB4510-03-1-A, J7 Conn_01x02_Pin, Q1 PMBT3904235, Q2 PMBT3904235, Q3 PMBT3904235, SW1 SW_Push, SW2 SW_Push, SW3 SW_Push, SW4 SW_Push, SW5 SW_Push, SW6 SW_Push, U1 NCP1117-3.3_SOT223, U2 ESP32-S2-SOLO, U3 CH340C

Commit message: Add changes for revision 0.2
Parts:
- removed R2: 10k, Resistor_SMD:R_0603_1608Metric, symbol Device:R
- added TP2: TestPoint, TestPoint:TestPoint_Pad_D1.5mm, symbol Connector:TestPoint
Connections:
- net BTN3: now also U2.15 (GPIO3/TOUCH3/ADC1_CH2); no longer U2.12 (GPIO8/TOUCH8/ADC1_CH7)
- net BTN4: now also U2.5 (GPIO5/TOUCH5/ADC1_CH4)
- net BTN5: now also U2.6 (GPIO6/TOUCH6/ADC1_CH5)
- net BTN6: now also U2.7 (GPIO7/TOUCH7/ADC1_CH6)
- net FXOS_INT1: now also TP3.1, U2.8 (GPIO15/U0RTS/ADC2_CH4/XTAL_32K_P)
- net FXOS_INT2: now also TP2.1
- net I2C_SCL: now also U2.12 (GPIO8/TOUCH8/ADC1_CH7)
- net I2C_SDA: now also U2.11 (GPIO18/U1RXD/ADC2_CH7/DAC_2/CLK_OUT3)
- net LED1: now also U2.13 (GPIO19/U1RTS/ADC2_CH8/CLK_OUT2/USB_D-); no longer U2.15 (GPIO3/TOUCH3/ADC1_CH2)
- net LED2: now also U2.14 (GPIO20/U1CTS/ADC2_CH9/CLK_OUT1/USB_D+); no longer U2.13 (GPIO19/U1RTS/ADC2_CH8/CLK_OUT2/USB_D-)
- net LEDS_DATA: now also U2.4 (GPIO4/TOUCH4/ADC1_CH3); no longer TP3.1, U2.8 (GPIO15/U0RTS/ADC2_CH4/XTAL_32K_P)
Other:
- note removed: "Agujeros de 3, no de 3,2"
- note removed: "NOTE 1"
- note removed: "NOTE 1: GPIO18 works as U1RXD and is in floating state when the chip is powered on, which may affect the chip's entry into download boot mode. To solve this issue, add an external pull-up resistor. TODO: revisar esto. Afecta a la UART 0?"
- note removed: "New HW requirements: - PCB adaptada a diana Decathlon (agujeros de sujección, botones, USB) - USB con datos y USB/UART - Botones: next_player, config (create AP), back, LEDs ON/OFF. TH? Tipo? - Buzzer? - LEDs bien colocados. Trough Hole? En recuadro pantalla. Con conector JST - Quitar resistencias, PU/PD, conectores solo donde debe haber, solo pines necesarios"
- moved on the sheet: BZ1, C1, C10, C11, C3, C4, C5, C6, C7, C8, C9, D1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
